File: Controller-2560/schematics/MidiController/mainboard.sch (EAGLE design)
At the start: 16 parts, among them IC1 74AC04N

Commit message: updated schematic
Parts:
- removed R7: 1k, SparkFun-Resistors:RESISTORAXIAL-0.3
- added C2: (no value), rcl:C-EU025-025X050
- added C3: (no value), rcl:CPOL-EUE1.8-4
- added DIS1: HD-K121, display-hp:HD-K121
- added IC2: MAX7219CNG, maxim:MAX7219CNG
- added J4: (no value), SparkFun-Connectors:CONN_02
- added J5: (no value), SparkFun-Connectors:CONN_03
- R6: value 1k -> (none)
Connections:
- new net N$13: IC2.ISET, R6.2
- new net N$14: DIS1.A1, DIS1.A2, IC2.SEGA
- new net N$15: DIS1.B1, DIS1.B2, IC2.SEGB
- new net N$16: DIS1.C1, DIS1.C2, IC2.SEGC
- new net N$17: DIS1.D1, DIS1.D2, IC2.SEGD
- new net N$18: DIS1.E1, DIS1.E2, IC2.SEGE
- new net N$19: DIS1.F1, DIS1.F2, IC2.SEGF
- new net N$20: DIS1.G1, DIS1.G2, IC2.SEGG
- new net N$23: DIS1.DP1, DIS1.DP2, IC2.SEGDP
- new net N$25: DIS1.CA1, IC2.DIG0
- new net N$26: DIS1.CA2, IC2.DIG1
- net +5V: now also C2.1, C3.+, IC1P.VCC, IC2.VCC, J4.2, R6.1
- net GND: now also C2.2, C3.-, IC1P.GND, IC2.GND@1, IC2.GND@2, J4.1; no longer R6.2, R7.2
- net N$8: no longer R6.1
- net N$9: no longer R7.1
- net RX3: now also J5.1
- net RX4: now also J5.2
- net TX4: now also J5.3
Other:
- moved on the sheet: R6
